File: hardware/london-underground-pcb.kicad_pcb (KiCad board)
At the start: 2 copper layers, 340 x 220 mm, 663 parts, among them SW1 TS-1187A-B-A-B, SW2 TS-1187A-B-A-B, SW3 TS-1187A-B-A-B, SW4 TS-1187A-B-A-B, U1 XIAO-RP2040-DIP

Commit message: Added bird logo to the back panel
Parts:
- added ? (x4): , Graphics, F.Cu at (8.30, -3.60)
- added ? (x4): , Graphics, F.Cu at (-14.5, 167.3)
- added ? (x4): , Graphics, F.Cu at (43.0, 233.0)
- added ?: , Graphics, F.Cu at (10.4, 176.2)
- added ?: , Graphics, F.Cu at (70.2, 216.5)
- added ?: , Graphics, B.Cu at (-14.5, 167.3)
- added ?: , Graphics, B.Cu at (8.30, -3.60)
- added ? (x5): , Graphics, B.Cu at (10.4, 176.2)
- added ? (x4): , Graphics, B.Cu at (70.2, 216.5)
- added ?: , Graphics, B.Cu at (43.0, 233.0)
- added ?: , Graphics, B.Cu at (334.0, -2.21)
- GND: renamed from ?; value (none) -> GND
Routing:
- net GND: vias 106 -> 109
Other:
- board text added: "+5V"
- board text added: "GND"
- board text added: "LED"
- board text added: "SW1"
- board text added: "SW2"
- board text added: "SW3"
- board text added: "SW4"
