File: hardware/london-underground-pcb.kicad_pcb (KiCad board)
At the start: 2 copper layers, 312 x 208 mm, 718 parts, among them SW1 TS-1187A-B-A-B, SW2 TS-1187A-B-A-B, SW3 TS-1187A-B-A-B, SW4 TS-1187A-B-A-B, U1 XIAO-RP2040-DIP

Commit message: submitted to JLCPCB 2025-Nov-30
Other:
- board text added: "https://github.com/funvill/London-Underground-PCB Created by: Steven Smethurst (@Funvill) Version: 2025-Nov-30"
- board text removed: "https://github.com/funvill/London-Underground-PCB Created by: Steven Smethurst (@Funvill) Version: 2025-Nov-25"
Changed lines of the file:
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@@
 		(sheetname "/")
 		(sheetfile "london-underground-pcb.kicad_sch")
+		(attr dnp)
 		(fp_line
 			(start -8.835 -8.513)
@@
 		)
 	)
-	(gr_text "https://github.com/funvill/London-Underground-PCB\nCreated by: Steven Smethurst (@Funvill)\nVersion: 2025-Nov-25"
+	(gr_text "https://github.com/funvill/London-Underground-PCB\nCreated by: Steven Smethurst (@Funvill)\nVersion: 2025-Nov-30"
 		(at 299.1 187.5 0)
 		(layer "B.SilkS")
